File: prj-kicad/pmod-mdb.sch (KiCad schematic (older format))
At the start: 14 parts, among them P1 PMOD, P2 MDB_P, U1 TLP185, U2 TLP185, U3 SN74LVC1G17, U4 SN74LVC1G17

Commit message: = ADD: Generate netlist and create first board routing
Parts:
- C1, D1: footprint (none) -> pmod-mdb:SMD0805
- C2, C3, R1, R2, R3, R4: footprint (none) -> pmod-mdb:SMD0603
- P1: footprint (none) -> pmod-mdb:CONN_PMOD-Male
- P2: footprint (none) -> pmod-mdb:CONN_64900621122
- U1, U2: footprint MFSOP-6 -> pmod-mdb:SOP6-4
- U3, U4: footprint (none) -> pmod-mdb:SOT23-5
Connections:
- net GND: no longer D1.2 (K)
- net GNDBUS: now also D1.2 (K)
Changed lines of the file:
@@
 EESchema Schematic File Version 4
-EELAYER 30 0
+LIBS:pmod-mdb-cache
+EELAYER 26 0
 EELAYER END
 $Descr A4 11693 8268
@@
 F 0 "P1" H 2350 3700 60  0000 C CNN
 F 1 "PMOD" H 2300 3000 60  0000 C CNN
-F 2 "" H 2550 3350 60  0000 C CNN
+F 2 "pmod-mdb:CONN_PMOD-Male" H 2550 3350 60  0001 C CNN
 F 3 "" H 2550 3350 60  0000 C CNN
 	1    2550 3350
@@
 $EndComp
 $Comp
-L pmod-mdb:VCC #PWR?
+L pmod-mdb:VCC #PWR0101
 U 1 1 5EA0372A
 P 2550 2850
-F 0 "#PWR?" H 2550 2810 30  0001 C CNN
+F 0 "#PWR0101" H 2550 2810 30  0001 C CNN
 F 1 "VCC" H 2559 2988 30  0000 C CNN
 F 2 "" H 2550 2850 60  0000 C CNN
@@
 Connection ~ 2550 2900
 $Comp
-L pmod-mdb:GND #PWR?
+L pmod-mdb:GND #PWR0102
 U 1 1 5EA03770
 P 2500 3800
-F 0 "#PWR?" H 2500 3800 30  0001 C CNN
+F 0 "#PWR0102" H 2500 3800 30  0001 C CNN
 F 1 "GND" H 2500 3730 30  0001 C CNN
 F 2 "" H 2500 3800 60  0000 C CNN
@@
 $EndComp
 $Comp
-L pmod-mdb:GND #PWR?
+L pmod-mdb:GND #PWR0103
 U 1 1 5EA03795
 P 2600 3800
-F 0 "#PWR?" H 2600 3800 30  0001 C CNN
+F 0 "#PWR0103" H 2600 3800 30  0001 C CNN
 F 1 "GND" H 2600 3730 30  0001 C CNN
 F 2 "" H 2600 3800 60  0000 C CNN
@@
 F 0 "P2" H 8300 3700 50  0000 C CNN
 F 1 "MDB_P" H 8300 3000 50  0000 C CNN
-F 2 "" H 8300 3350 60  0000 C CNN
+F 2 "pmod-mdb:CONN_64900621122" H 8300 3350 60  0001 C CNN
 F 3 "" H 8300 3350 60  0000 C CNN
 	1    8300 3350
@@
 $EndComp
 $Comp
-L pmod-mdb:GNDBUS #PWR?
+L pmod-mdb:GNDBUS #PWR0104
 U 1 1 5EA03F4C
 P 8750 3700
-F 0 "#PWR?" H 8750 3550 50  0001 C CNN
+F 0 "#PWR0104" H 8750 3550 50  0001 C CNN
 F 1 "GNDBUS" H 8750 3600 50  0001 C CNN
 F 2 "" H 8750 3700 50  0000 C CNN
@@
 	8750 3500 8650 3500
 $Comp
-L pmod-mdb:GNDBUS #PWR?
+L pmod-mdb:GNDBUS #PWR0105
 U 1 1 5EA04006
 P 7850 3700
-F 0 "#PWR?" H 7850 3550 50  0001 C CNN
+F 0 "#PWR0105" H 7850 3550 50  0001 C CNN
 F 1 "GNDBUS" H 7850 3600 50  0001 C CNN
 F 2 "" H 7850 3700 50  0000 C CNN
@@
 F 0 "U1" H 6300 3000 50  0000 C CNN
 F 1 "TLP185" H 6300 2550 50  0000 C CNN
-F 2 "MFSOP-6" H 6300 3075 50  0001 C CIN
+F 2 "pmod-mdb:SOP6-4" H 6300 3075 50  0001 C CIN
 F 3 "http://www.semicon.toshiba.co.jp/docs/datasheet/en/Opto/TLP185_en_datasheet_120214.pdf" H 6300 2984 50  0001 C CNN
 	1    6300 2750
@@
 F 0 "U2" H 6300 4150 50  0000 C CNN
 F 1 "TLP185" H 6300 3700 50  0000 C CNN
-F 2 "MFSOP-6" H 6300 4225 50  0001 C CIN
+F 2 "pmod-mdb:SOP6-4" H 6300 4225 50  0001 C CIN
 F 3 "http://www.semicon.toshiba.co.jp/docs/datasheet/en/Opto/TLP185_en_datasheet_120214.pdf" H 6300 4134 50  0001 C CNN
 	1    6300 3900
@@
 $EndComp
 $Comp
-L pmod-mdb:GNDBUS #PWR?
+L pmod-mdb:GNDBUS #PWR0106
 U 1 1 5EA04894
 P 6700 2950
-F 0 "#PWR?" H 6700 2800 50  0001 C CNN
+F 0 "#PWR0106" H 6700 2800 50  0001 C CNN
 F 1 "GNDBUS" H 6700 2850 50  0001 C CNN
 F 2 "" H 6700 2950 50  0000 C CNN
@@
 	6700 2850 6600 2850
 $Comp
-L pmod-mdb:GNDBUS #PWR?
+L pmod-mdb:GNDBUS #PWR0107
 U 1 1 5EA04E7F
 P 6700 4100
-F 0 "#PWR?" H 6700 3950 50  0001 C CNN
+F 0 "#PWR0107" H 6700 3950 50  0001 C CNN
 F 1 "GNDBUS" H 6700 4000 50  0001 C CNN
 F 2 "" H 6700 4100 50  0000 C CNN
@@
 F 0 "R1" V 6850 3800 50  0000 C CNN
 F 1 "1k" V 6950 3800 45  0000 C CNN
-F 2 "" H 6950 3800 60  0000 C CNN
+F 2 "pmod-mdb:SMD0603" H 6950 3800 60  0001 C CNN
 F 3 "" H 6950 3800 60  0000 C CNN
 	1    6950 3800
@@
 	7450 3350 7450 3800
 $Comp
-L pmod-mdb:GND #PWR?
+L pmod-mdb:GND #PWR0108
 U 1 1 5EA05EB3
 P 5900 2950
-F 0 "#PWR?" H 5900 2950 30  0001 C CNN
+F 0 "#PWR0108" H 5900 2950 30  0001 C CNN
 F 1 "GND" H 5900 2880 30  0001 C CNN
 F 2 "" H 5900 2950 60  0000 C CNN
@@
 	5900 4000 6000 4000
 $Comp
-L pmod-mdb:GND #PWR?
+L pmod-mdb:GND #PWR0109
 U 1 1 5EA06453
 P 5900 4100
-F 0 "#PWR?" H 5900 4100 30  0001 C CNN
+F 0 "#PWR0109" H 5900 4100 30  0001 C CNN
 F 1 "GND" H 5900 4030 30  0001 C CNN
 F 2 "" H 5900 4100 60  0000 C CNN
@@
 F 0 "R2" V 5450 2650 50  0000 C CNN
 F 1 "330" V 5550 2650 45  0000 C CNN
-F 2 "" H 5550 2650 60  0000 C CNN
+F 2 "pmod-mdb:SMD0603" H 5550 2650 60  0001 C CNN
 F 3 "" H 5550 2650 60  0000 C CNN
 	1    5550 2650
@@
 F 0 "R3" V 5450 3600 50  0000 C CNN
 F 1 "10k" V 5550 3600 45  0000 C CNN
-F 2 "" H 5550 3600 60  0000 C CNN
+F 2 "pmod-mdb:SMD0603" H 5550 3600 60  0001 C CNN
 F 3 "" H 5550 3600 60  0000 C CNN
 	1    5550 3600
@@
 $EndComp
 $Comp
-L pmod-mdb:VCC #PWR?
+L pmod-mdb:VCC #PWR0110
 U 1 1 5EA06A41
 P 5900 3500
-F 0 "#PWR?" H 5900 3460 30  0001 C CNN
+F 0 "#PWR0110" H 5900 3460 30  0001 C CNN
 F 1 "VCC" H 5909 3638 30  0000 C CNN
 F 2 "" H 5900 3500 60  0000 C CNN
@@
 F 0 "U3" H 4650 2900 50  0000 L CNN
 F 1 "SN74LVC1G17" H 4700 2600 40  0000 L CNN
-F 2 "" H 4600 2750 50  0001 C CNN
+F 2 "pmod-mdb:SOT23-5" H 4600 2750 50  0001 C CNN
 F 3 "" H 4600 2750 50  0001 C CNN
 	1    4600 2750
@@
 	5050 2650 5300 2650
 $Comp
-L pmod-mdb:VCC #PWR?
+L pmod-mdb:VCC #PWR0111
 U 1 1 5EA08959
 P 4600 2550
-F 0 "#PWR?" H 4600 2510 30  0001 C CNN
+F 0 "#PWR0111" H 4600 2510 30  0001 C CNN
 F 1 "VCC" H 4609 2688 30  0000 C CNN
 F 2 "" H 4600 2550 60  0000 C CNN
@@
 $EndComp
 $Comp
-L pmod-mdb:GND #PWR?
+L pmod-mdb:GND #PWR0112
 U 1 1 5EA0899A
 P 4600 2950
-F 0 "#PWR?" H 4600 2950 30  0001 C CNN
+F 0 "#PWR0112" H 4600 2950 30  0001 C CNN
 F 1 "GND" H 4600 2880 30  0001 C CNN
 F 2 "" H 4600 2950 60  0000 C CNN
@@
 F 0 "U4" H 4550 4050 50  0000 R CNN
 F 1 "SN74LVC1G17" H 4500 3750 40  0000 R CNN
-F 2 "" H 4600 3900 50  0001 C CNN
+F 2 "pmod-mdb:SOT23-5" H 4600 3900 50  0001 C CNN
 F 3 "" H 4600 3900 50  0001 C CNN
 	1    4600 3900
@@
 $EndComp
 $Comp
-L pmod-mdb:VCC #PWR?
+L pmod-mdb:VCC #PWR0113
 U 1 1 5EA097C0
 P 4600 3700
-F 0 "#PWR?" H 4600 3660 30  0001 C CNN
+F 0 "#PWR0113" H 4600 3660 30  0001 C CNN
 F 1 "VCC" H 4609 3838 30  0000 C CNN
 F 2 "" H 4600 3700 60  0000 C CNN
@@
 	4600 4100 4600 4050
 $Comp
-L pmod-mdb:GND #PWR?
+L pmod-mdb:GND #PWR0114
 U 1 1 5EA0A63E
 P 4600 4100
-F 0 "#PWR?" H 4600 4100 30  0001 C CNN
+F 0 "#PWR0114" H 4600 4100 30  0001 C CNN
 F 1 "GND" H 4600 4030 30  0001 C CNN
 F 2 "" H 4600 4100 60  0000 C CNN
@@
 F 0 "C1" H 2700 4600 50  0000 L CNN
 F 1 "10uF" H 2700 4400 50  0000 L CNN
-F 2 "" H 2650 4500 60  0000 C CNN
+F 2 "pmod-mdb:SMD0805" H 2650 4500 60  0001 C CNN
 F 3 "" H 2650 4500 60  0000 C CNN
 	1    2650 4500
@@
 $EndComp
 $Comp
-L pmod-mdb:VCC #PWR?
+L pmod-mdb:VCC #PWR0115
 U 1 1 5EA051BB
 P 2550 4200
-F 0 "#PWR?" H 2550 4160 30  0001 C CNN
+F 0 "#PWR0115" H 2550 4160 30  0001 C CNN
 F 1 "VCC" H 2559 4338 30  0000 C CNN
 F 2 "" H 2550 4200 60  0000 C CNN
@@
 $EndComp
 $Comp
-L pmod-mdb:GND #PWR?
+L pmod-mdb:GND #PWR0116
 U 1 1 5EA05D41
 P 2650 4750
-F 0 "#PWR?" H 2650 4750 30  0001 C CNN
+F 0 "#PWR0116" H 2650 4750 30  0001 C CNN
 F 1 "GND" H 2650 4680 30  0001 C CNN
 F 2 "" H 2650 4750 60  0000 C CNN
@@
 F 0 "C2" H 3000 4600 50  0000 L CNN
 F 1 "100nF" H 3000 4400 50  0000 L CNN
-F 2 "" H 2950 4500 60  0000 C CNN
+F 2 "pmod-mdb:SMD0603" H 2950 4500 60  0001 C CNN
 F 3 "" H 2950 4500 60  0000 C CNN
 	1    2950 4500
@@
 F 0 "C3" H 3300 4600 50  0000 L CNN
 F 1 "100nF" H 3300 4400 50  0000 L CNN
-F 2 "" H 3250 4500 60  0000 C CNN
+F 2 "pmod-mdb:SMD0603" H 3250 4500 60  0001 C CNN
 F 3 "" H 3250 4500 60  0000 C CNN
 	1    3250 4500
@@
 $EndComp
 $Comp
-L pmod-mdb:GND #PWR?
+L pmod-mdb:GND #PWR0117
 U 1 1 5EA0723D
 P 2950 4750
-F 0 "#PWR?" H 2950 4750 30  0001 C CNN
+F 0 "#PWR0117" H 2950 4750 30  0001 C CNN
 F 1 "GND" H 2950 4680 30  0001 C CNN
 F 2 "" H 2950 4750 60  0000 C CNN
@@
 $EndComp
 $Comp
-L pmod-mdb:GND #PWR?
+L pmod-mdb:GND #PWR0118
 U 1 1 5EA074F8
 P 3250 4750
-F 0 "#PWR?" H 3250 4750 30  0001 C CNN
+F 0 "#PWR0118" H 3250 4750 30  0001 C CNN
 F 1 "GND" H 3250 4680 30  0001 C CNN
 F 2 "" H 3250 4750 60  0000 C CNN
@@
 Connection ~ 2950 4250
 $Comp
-L pmod-mdb:VBus #PWR?
+L pmod-mdb:VBus #PWR0119
 U 1 1 5EA0F35B
 P 8750 3100
-F 0 "#PWR?" H 8750 3060 30  0001 C CNN
+F 0 "#PWR0119" H 8750 3060 30  0001 C CNN
 F 1 "VBus" H 8759 3238 30  0000 C CNN
 F 2 "" H 8750 3100 60  0000 C CNN
@@
 	8750 3200 8650 3200
 $Comp
-L pmod-mdb:VBus #PWR?
+L pmod-mdb:VBus #PWR0120
 U 1 1 5EA10CBF
 P 7650 4400
-F 0 "#PWR?" H 7650 4360 30  0001 C CNN
+F 0 "#PWR0120" H 7650 4360 30  0001 C CNN
 F 1 "VBus" H 7659 4538 30  0000 C CNN
 F 2 "" H 7650 4400 60  0000 C CNN
@@
 F 0 "R4" V 7900 4500 50  0000 C CNN
 F 1 "2,4k" V 8000 4500 45  0000 C CNN
-F 2 "" H 8000 4500 60  0000 C CNN
+F 2 "pmod-mdb:SMD0603" H 8000 4500 60  0001 C CNN
 F 3 "" H 8000 4500 60  0000 C CNN
 	1    8000 4500
@@
 F 0 "D1" H 8550 4600 50  0000 C CNN
 F 1 "LED" H 8550 4400 25  0000 C CNN
-F 2 "" H 8550 4500 60  0000 C CNN
+F 2 "pmod-mdb:SMD0805" H 8550 4500 60  0001 C CNN
 F 3 "" H 8550 4500 60  0000 C CNN
 	1    8550 4500
-	1    0    0    -1
-$EndComp
-$Comp
-L pmod-mdb:GND #PWR?
-U 1 1 5EA16E6C
-P 8850 4600
-F 0 "#PWR?" H 8850 4600 30  0001 C CNN
-F 1 "GND" H 8850 4530 30  0001 C CNN
-F 2 "" H 8850 4600 60  0000 C CNN
-F 3 "" H 8850 4600 60  0000 C CNN
-	1    8850 4600
 	1    0    0    -1
 $EndComp
@@
 Text Notes 5950 5100 0    50   ~ 0
 Galvanic isolation
+$Comp
+L pmod-mdb:GNDBUS #PWR0121
+U 1 1 5EA1A0E2
+P 8850 4600
+F 0 "#PWR0121" H 8850 4450 50  0001 C CNN
+F 1 "GNDBUS" H 8854 4674 50  0001 C CNN
+F 2 "" H 8850 4600 50  0000 C CNN
+F 3 "" H 8850 4600 50  0000 C CNN
+	1    8850 4600
+	1    0    0    -1
+$EndComp
 $EndSCHEMATC
